File: hardware/electrical/solarboard/solarboard.kicad_pcb (KiCad board)
At the start: 2 copper layers, 10 parts, among them J1 Conn_01x02_Pin

Commit message: revision solar board
Parts:
- moved J1 30.0 mm to (107.0, 175.9)
- moved U3 24.8 mm to (40.0, 142.1)
- moved U6 24.8 mm to (107.1, 142.1)
- moved U9 24.8 mm to (174.2, 142.1)
- moved U4 24.8 mm to (107.1, 7.90)
- moved U5 24.8 mm to (107.1, 75.0)
- moved U7 24.8 mm to (174.2, 7.90)
- moved U8 24.8 mm to (174.2, 75.0)
- moved U1 24.8 mm to (40.0, 7.90)
- moved U2 24.8 mm to (40.0, 75.0)
Routing:
- net Net-(J1-Pin_2): track 632.9 -> 581.7 mm
- removed copper zone on F.Cu, net (none)

Commit message: update designs and firmware
Parts:
- moved J1 0.06 mm to (107.0, 175.9)
- moved U1 0.06 mm to (40.0, 7.87)
- moved U4 0.06 mm to (107.0, 7.87)
- moved U2 0.06 mm to (40.0, 75.0)
- moved U5 0.06 mm to (107.0, 75.0)
- moved U3 0.06 mm to (40.0, 142.1)
- moved U6 0.06 mm to (107.0, 142.1)
- moved U7 0.06 mm to (174.2, 7.87)
- moved U8 0.06 mm to (174.2, 75.0)
- moved U9 0.06 mm to (174.2, 142.1)
Routing:
- net Net-(J1-Pin_2): track 581.7 -> 636.2 mm
